Commit message: Added version with and without urdf panda inertial link values

File: test_frite_with_mocap/DDPG_GPU_MPI/gym_panda_frite/envs/urdf/franka_panda/panda_without_intertial.urdf (robot description, URDF)
Before this commit: robot panda, 13 links, 12 joints
Links:
- link panda_hand: mass .81 -> None
- link panda_hand_tcp: mass 0 -> None
- link panda_leftfinger: mass 0.1 -> None
- link panda_link0: mass 2.9 -> None
- link panda_link1: mass 2.7 -> None
- link panda_link2: mass 2.73 -> None
- link panda_link3: mass 2.04 -> None
- link panda_link4: mass 2.08 -> None
- link panda_link5: mass 3 -> None
- link panda_link6: mass 1.3 -> None
- link panda_link7: mass .2 -> None
- link panda_link8: mass 0.0 -> None
- link panda_rightfinger: mass 0.1 -> None
